Commit message: Fixed Orientation

File: urdf/planar_3dof.urdf (robot description, URDF)
Before this commit: robot planar_3dof, 76 links, 75 joints
Joints:
- joint AdductionshoulderL: limit lower=0.349066 upper=2.87979 effort=1 velocity=20 -> lower=-0.724 upper=1.97979 effort=1 velocity=20
- joint HandFelxionR: limit lower=-0.174533 upper=0.523599 effort=1 velocity=20 -> lower=-0.274533 upper=0.523599 effort=1 velocity=20
- joint abductionShoulderR: limit lower=-2.87979 upper=-0.349066 effort=1 velocity=20 -> lower=0.568 upper=-0.949066 effort=1 velocity=20
